File: EL_Electrical/timer/hardware/timer_controller.sch (EAGLE design)
At the start: 20 parts, among them IC2 TC4S584F, IC3 TC4S584F, IC4 LM555D, Q1 BSS138, T1 2N2369

Commit message: Update sch and PCB (Timer Controller)
Parts:
- added BASE_NPN: BASE_NPN, pinhead:PINHD-1X1
- added GATE_MOSFET: GATE_MOSFET, pinhead:PINHD-1X1
- added J1: 22-27-2041-04, con-molex:22-27-2041-04
- added OUT: OUT, pinhead:PINHD-1X1
- added TRIGGER: TRIGGER, pinhead:PINHD-1X1
- C2: value 200µF -> 22µF
- R2: value 1.8k -> 18k
- R5: value 1.2k -> 12k
Connections:
- removed net N$19: R5.1, R7.2, T1.C
- removed net N$21: IC2A.O, R3.1, R7.1
- removed net N$23: C4.2, C5.2
- removed net N$24: IC2A.I, IC4.Q
- removed net N$25: IC3A.O, R8.2
- new net BASE_NPN: BASE_NPN.1, IC3A.O, R8.2
- new net GATE_MOSFET: GATE_MOSFET.1, IC2A.O, R3.1, R7.1
- new net N$2: R9.1, T1.C
- new net OUT: IC2A.I, IC4.Q, OUT.1
- net +12V: now also IC2P.VCC, IC3P.VCC, J1-1.S
- net BP_START: now also J1-3.S
- net GND: now also C4.2, C5.2, IC2P.GND, IC3P.GND, J1-4.S
- net N$26: now also R5.1, R7.2; no longer R9.1
- net RELAIS_INJECTEUR: now also J1-2.S
- net TRIGGER: now also TRIGGER.1
Other:
- note removed: "FSG 2019 BSPD V 0.2"
- moved on the sheet: IC2, IC3, R10, R4, R7, R8, R9, T1
