File: EL_Electrical/timer/hardware/timer_controller.sch (EAGLE design)
At the start: 25 parts, among them IC2 TC4S584F, IC3 TC4S584F, IC4 LM555D, J1 22-27-2041-04, Q1 BSS138, T1 2N2369

Commit message: Change footprint for 150uF capacitor. Rearrange text infos. Add a GND test pin
Parts:
- added GND: GND, pinhead:PINHD-1X1
- C2: device rcl:C-EUC0805 -> rcl:CPOL-EU153CLV-0605
Connections:
- net GND: now also C2.-, GND.1; no longer C2.2
- net TRIGGER: now also C2.+; no longer C2.1
Changed lines of the file:
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@@
 <?xml version="1.0" encoding="utf-8"?>
 <!DOCTYPE eagle SYSTEM "eagle.dtd">
-<eagle version="9.5.2">
+<eagle version="9.5.1">
 <drawing>
 <settings>
@@
 <part name="FRAME1" library="frames" deviceset="A4L-LOC" device=""/>
 <part name="C1" library="rcl" library_urn="urn:adsk.eagle:library:334" deviceset="C-EU" device="C0805" package3d_urn="urn:adsk.eagle:package:23617/2" value="2.2µF"/>
-<part name="C2" library="rcl" library_urn="urn:adsk.eagle:library:334" deviceset="C-EU" device="C0805" package3d_urn="urn:adsk.eagle:package:23617/2" value="150µF"/>
+<part name="C2" library="rcl" library_urn="urn:adsk.eagle:library:334" deviceset="CPOL-EU" device="153CLV-0605" package3d_urn="urn:adsk.eagle:package:23398/2" value="150µF"/>
 <part name="C3" library="rcl" library_urn="urn:adsk.eagle:library:334" deviceset="C-EU" device="C0805" package3d_urn="urn:adsk.eagle:package:23617/2" value="0.01µF"/>
 <part name="R1" library="rcl" library_urn="urn:adsk.eagle:library:334" deviceset="R-EU_" device="R0805" package3d_urn="urn:adsk.eagle:package:23553/2" value="2.2k"/>
@@
 <part name="P+5" library="supply1" library_urn="urn:adsk.eagle:library:371" deviceset="+12V" device=""/>
 <part name="GND3" library="supply1" library_urn="urn:adsk.eagle:library:371" deviceset="GND" device=""/>
+<part name="GND" library="pinhead" library_urn="urn:adsk.eagle:library:325" deviceset="PINHD-1X1" device="" package3d_urn="urn:adsk.eagle:package:22485/2" value="GND"/>
+<part name="GND4" library="supply1" library_urn="urn:adsk.eagle:library:371" deviceset="GND" device=""/>
 </parts>
 <sheets>
@@
 <attribute name="NAME" x="116.205" y="78.105" size="1.778" layer="95"/>
 </instance>
+<instance part="GND" gate="G$1" x="167.64" y="45.72" smashed="yes">
+<attribute name="NAME" x="161.29" y="48.895" size="1.778" layer="95"/>
+<attribute name="VALUE" x="161.29" y="40.64" size="1.778" layer="96"/>
+</instance>
+<instance part="GND4" gate="1" x="152.4" y="43.18" smashed="yes">
+<attribute name="VALUE" x="149.86" y="40.64" size="1.778" layer="96"/>
+</instance>
 </instances>
 <busses>
@@
 <pinref part="GND26" gate="1" pin="GND"/>
 <wire x1="160.02" y1="96.52" x2="160.02" y2="99.06" width="0.1524" layer="91"/>
-<pinref part="C2" gate="G$1" pin="2"/>
+<pinref part="C2" gate="G$1" pin="-"/>
 <wire x1="165.1" y1="101.6" x2="165.1" y2="99.06" width="0.1524" layer="91"/>
 <pinref part="R2" gate="G$1" pin="1"/>
@@
 <pinref part="GND3" gate="1" pin="GND"/>
 <wire x1="119.38" y1="71.12" x2="119.38" y2="68.58" width="0.1524" layer="91"/>
+</segment>
+<segment>
+<pinref part="GND" gate="G$1" pin="1"/>
+<pinref part="GND4" gate="1" pin="GND"/>
+<wire x1="165.1" y1="45.72" x2="152.4" y2="45.72" width="0.1524" layer="91"/>
 </segment>
 </net>
@@
 <segment>
 <wire x1="167.64" y1="116.84" x2="165.1" y2="116.84" width="0.1524" layer="91"/>
-<pinref part="C2" gate="G$1" pin="1"/>
+<pinref part="C2" gate="G$1" pin="+"/>
 <wire x1="165.1" y1="109.22" x2="165.1" y2="116.84" width="0.1524" layer="91"/>
 <junction x="165.1" y="109.22"/>
@@
 packages will not be understood (or retained) with this version.
 </note>
+<note version="8.4" severity="warning">
+Since Version 8.4, EAGLE supports properties for SPICE simulation.
+Probes in schematics and SPICE mapping objects found in parts and library devices
+will not be understood with this version. Update EAGLE to the latest version
+for full support of SPICE simulation.
+</note>
 </compatibility>

Commit message: Timer_controller add pin
Parts:
- removed J1: 22-27-2041-04, con-molex:22-27-2041-04
- added J_TX_CAN2: (no value), jumper:JP2E
- added X1: 22-23-2051, con-molex:22-23-2051
Connections:
- new net 12_SWITCHES: J_TX_CAN2.3, X1-1.S
- new net RELAIS_INJECTEUR_12_PROTEGE: D1.C, J_TX_CAN2.2
- new net RELAIS_INJECTEUR_MASSE: D1.A, Q1.D
- net +12V: now also J_TX_CAN2.1, X1-2.S; no longer D1.C, J1-1.S
- net BP_START: now also X1-4.S; no longer J1-3.S
- net GND: now also X1-5.S; no longer J1-4.S
- net RELAIS_INJECTEUR: now also X1-3.S; no longer D1.A, J1-2.S, Q1.D
