File: EL_Electrical/timer/hardware/timer_controller_V2.brd (EAGLE design)
At the start: 44 x 36 mm, 27 parts, among them IC2 TC4S584F, IC3 TC4S584F, IC4 LM555D, Q1 BSS138, T1 2N2369, X1 22-23-2051

Commit message: Timer - production files
Parts:
- removed R7: 100, rcl:R0805
- added IC1: TC4S584F, 74xx-little-us:SOT23-5
- added IC5: Gate OR, 74xx-little-us:SOT23-5
- moved R5 12.3 mm to (18.8, 30.7), turned to 0 degrees
- moved TRIGGER 6.44 mm to (21.6, 25.6)
- moved GATE_MOSFET 5.96 mm to (21.1, 6.50)
- moved C2 5.07 mm to (26.5, 30.6), turned to 180 degrees
- moved R2 4.78 mm to (28.4, 25.0), turned to 180 degrees
- moved IC2 3.67 mm to (26.9, 11.9)
- moved OUT 2.70 mm to (26.3, 18.4)
Connections:
- new net N$3: IC1.4, IC5.2
- new net N$4: IC2.4, IC5.1
- net +12V: now also IC1.5, IC5.5
- net BASE_NPN: now also IC1.2
- net GATE_MOSFET: now also IC5.4; no longer IC2.4, R7.1
- net GND: now also IC1.3, IC5.3
- net N$26: no longer R7.2
Routing:
- net N$26: track 19.4 -> 3.50 mm
- net +12V: track 47.5 -> 58.7 mm, vias 4 -> 1
- net BASE_NPN: track 4.45 -> 11.7 mm
- net TRIGGER: track 18.3 -> 24.8 mm
- net N$3: track 0.00 -> 5.46 mm
- net N$4: track 0.00 -> 4.08 mm
- net GATE_MOSFET: track 8.16 -> 11.2 mm
- net OUT: track 10.3 -> 13.0 mm
Other:
- board text added: "Timer INVICTUS v2.0"
- board text removed: "Timer INVICTUS"
