File: EL_Electrical/Gearshift/invictus/gearshift_controller.brd (EAGLE design)
At the start: 66.4 x 62.4 mm, 69 parts, among them IC1 MCP2562-E_SN, IC2 MCP2515-I_SO, Q1 BSS138, Q10 BSS138, Q2 BSS138, Q3 BSS138, Q4 BSS138, Q5 BSS138, Q6 BSS138, Q8 BSS138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

Commit message: Update holes and text
Parts:
- renumbered ALIM to POWER
Changed lines of the file:
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@@
 NEUTRE</text>
 <dimension x1="0.28" y1="0" x2="0.4" y2="62.36" x3="-7.38" y3="31.18" textsize="1.778" layer="47" dtype="vertical"/>
+<dimension x1="2.675" y1="59.8325" x2="63.4925" y2="59.8325" x3="33.08375" y3="70.64" textsize="1.778" layer="47" dtype="horizontal"/>
+<dimension x1="63.4925" y1="59.8325" x2="11.15" y2="73.88" x3="37.32125" y3="-3.46" textsize="1.778" layer="47" dtype="horizontal"/>
 </plain>
 <attributes>
@@
 <attribute name="MF" value="MOLEX" x="-5.6275" y="-19.685" size="1.778" layer="27" rot="R270" display="off"/>
 <attribute name="MPN" value="" x="-5.6275" y="-19.685" size="1.778" layer="27" rot="R270" display="off"/>
-<attribute name="NAME" x="4.2904" y="44.7549" size="1.016" layer="27" ratio="10" rot="R90"/>
+<attribute name="NAME" x="4.2904" y="44.2749" size="1.016" layer="27" ratio="10" rot="R90"/>
 <attribute name="OC_FARNELL" value="unknown" x="-5.6275" y="-19.685" size="1.778" layer="27" rot="R270" display="off"/>
 <attribute name="OC_NEWARK" value="unknown" x="-5.6275" y="-19.685" size="1.778" layer="27" rot="R270" display="off"/>
@@
 <attribute name="VALUE" x="48.3475" y="10.92" size="0.8128" layer="27" align="top-right"/>
 </element>
-<element name="ALIM" library="con-molex" library_urn="urn:adsk.eagle:library:165" package="6410-02" package3d_urn="urn:adsk.eagle:package:8078645/1" value="22-27-2021-02" x="8.2775" y="55.6475" smashed="yes" rot="R90">
+<element name="POWER" library="con-molex" library_urn="urn:adsk.eagle:library:165" package="6410-02" package3d_urn="urn:adsk.eagle:package:8078645/1" value="22-27-2021-02" x="8.2775" y="55.6475" smashed="yes" rot="R90">
 <attribute name="MF" value="MOLEX" x="8.2775" y="55.6475" size="1.778" layer="27" rot="R90" display="off"/>
 <attribute name="MPN" value="" x="8.2775" y="55.6475" size="1.778" layer="27" rot="R90" display="off"/>
-<attribute name="NAME" x="4.3204" y="53.5774" size="1.27" layer="27" ratio="10" rot="R90"/>
+<attribute name="NAME" x="4.2804" y="52.6574" size="1.016" layer="27" ratio="10" rot="R90"/>
 <attribute name="OC_FARNELL" value="unknown" x="8.2775" y="55.6475" size="1.778" layer="27" rot="R90" display="off"/>
 <attribute name="OC_NEWARK" value="unknown" x="8.2775" y="55.6475" size="1.778" layer="27" rot="R90" display="off"/>
@@
 <contactref element="C107" pad="1"/>
 <contactref element="C106" pad="1"/>
-<contactref element="ALIM" pad="2"/>
+<contactref element="POWER" pad="2"/>
 <wire x1="11.0625" y1="55.6625" x2="9.7775" y2="54.3775" width="0.8128" layer="1"/>
 <wire x1="8.2775" y1="54.3775" x2="9.7775" y2="54.3775" width="0.8128" layer="1"/>
@@
 <wire x1="15.875" y1="33.9725" x2="15.24" y2="33.3375" width="0.6096" layer="1"/>
 <wire x1="15.24" y1="30.8175" x2="15.5775" y2="30.48" width="0.6096" layer="1"/>
-<contactref element="ALIM" pad="1"/>
+<contactref element="POWER" pad="1"/>
 <wire x1="13.135" y1="57.5625" x2="13.02" y2="57.5625" width="0.6096" layer="1"/>
 <wire x1="13.02" y1="57.5625" x2="13.065" y2="57.5175" width="0.8128" layer="1"/>
